File: 6 Controller/SNES controller protoboard/SNES controller protoboard.kicad_pcb (KiCad board)
At the start: 2 copper layers, 128 x 52 mm, 920 parts, among them U1 Arduino_Pro_Micro

Commit message: Controller update and workshop cost update
Other:
- board text added: "DESIGN BY CM VAN RIET"
- board text added: "JLCJLCJLCJLC"
